Commit message: phase2_1

File: src/rice_weeding_description/urdf/rice_weeding_robot.urdf.xacro (robot description, xacro)
@@ -15,5 +15,5 @@
   <xacro:property name="body_center_z_value" value="${float(xacro.arg('body_center_z'))}"/>
   <xacro:property name="mast_length_value" value="${float(xacro.arg('sensor_height')) - float(xacro.arg('body_center_z'))}"/>
-  <material name="paddy_green"><color rgba="0.10 0.38 0.16 1.0"/></material>
+  <material name="body_black"><color rgba="0.03 0.03 0.03 1.0"/></material>
   <material name="sensor_black"><color rgba="0.04 0.05 0.04 1.0"/></material>
   <material name="cage_wheel_gray"><color rgba="0.22 0.24 0.22 1.0"/></material>
@@ -21,5 +21,5 @@
   <link name="base_link">
     <inertial><mass value="$(arg mass)"/><origin xyz="0 0 0"/><inertia ixx="3.0" ixy="0" ixz="0" iyy="3.0" iyz="0" izz="5.0"/></inertial>
-    <visual><geometry><box size="$(arg body_length) $(arg body_width) $(arg body_height)"/></geometry><material name="paddy_green"/></visual>
+    <visual><geometry><box size="$(arg body_length) $(arg body_width) $(arg body_height)"/></geometry><material name="body_black"/></visual>
     <collision><geometry><box size="$(arg body_length) $(arg body_width) $(arg body_height)"/></geometry></collision>
   </link>
@@ -31,4 +31,5 @@
     <link name="${name}_link">
       <visual><origin rpy="1.57079632679 0 0"/><geometry><cylinder radius="${wheel_radius_value}" length="$(arg wheel_width)"/></geometry><material name="cage_wheel_gray"/></visual>
+      <collision><origin rpy="1.57079632679 0 0"/><geometry><cylinder radius="${wheel_radius_value}" length="$(arg wheel_width)"/></geometry></collision>
     </link>
     <joint name="base_link_to_${name}" type="fixed">

Commit message: phase2_4

File: src/rice_weeding_description/urdf/rice_weeding_robot.urdf.xacro (robot description, xacro)
@@ -5,9 +5,17 @@
   <xacro:arg name="body_height" default="0.0"/>
   <xacro:arg name="body_center_z" default="0.0"/>
-  <xacro:arg name="mass" default="0.0"/>
+  <xacro:arg name="body_mass" default="0.0"/>
+  <xacro:arg name="wheel_mass" default="0.0"/>
   <xacro:arg name="wheel_diameter" default="0.0"/>
   <xacro:arg name="wheel_width" default="0.0"/>
+  <xacro:arg name="wheel_joint_damping" default="0.0"/>
+  <xacro:arg name="wheel_joint_friction" default="0.0"/>
   <xacro:arg name="track_width" default="0.0"/>
   <xacro:arg name="wheelbase" default="0.0"/>
+  <xacro:arg name="max_forward_velocity" default="0.0"/>
+  <xacro:arg name="max_reverse_velocity" default="0.0"/>
+  <xacro:arg name="max_angular_velocity" default="0.0"/>
+  <xacro:arg name="max_linear_acceleration" default="0.0"/>
+  <xacro:arg name="max_linear_deceleration" default="0.0"/>
   <xacro:arg name="sensor_height" default="0.0"/>
   <xacro:arg name="gnss_baseline" default="0.0"/>
@@ -15,4 +23,7 @@
   <xacro:property name="body_center_z_value" value="${float(xacro.arg('body_center_z'))}"/>
   <xacro:property name="mast_length_value" value="${float(xacro.arg('sensor_height')) - float(xacro.arg('body_center_z'))}"/>
+  <xacro:property name="wheel_mass_value" value="${float(xacro.arg('wheel_mass'))}"/>
+  <xacro:property name="wheel_transverse_inertia" value="${wheel_mass_value * (3.0 * wheel_radius_value * wheel_radius_value + float(xacro.arg('wheel_width')) * float(xacro.arg('wheel_width'))) / 12.0}"/>
+  <xacro:property name="wheel_axial_inertia" value="${0.5 * wheel_mass_value * wheel_radius_value * wheel_radius_value}"/>
   <material name="body_black"><color rgba="0.03 0.03 0.03 1.0"/></material>
   <material name="sensor_black"><color rgba="0.04 0.05 0.04 1.0"/></material>
@@ -20,5 +31,5 @@
   <link name="base_footprint"/>
   <link name="base_link">
-    <inertial><mass value="$(arg mass)"/><origin xyz="0 0 0"/><inertia ixx="3.0" ixy="0" ixz="0" iyy="3.0" iyz="0" izz="5.0"/></inertial>
+    <inertial><mass value="$(arg body_mass)"/><origin xyz="0 0 0"/><inertia ixx="3.0" ixy="0" ixz="0" iyy="3.0" iyz="0" izz="5.0"/></inertial>
     <visual><geometry><box size="$(arg body_length) $(arg body_width) $(arg body_height)"/></geometry><material name="body_black"/></visual>
     <collision><geometry><box size="$(arg body_length) $(arg body_width) $(arg body_height)"/></geometry></collision>
@@ -30,10 +41,17 @@
   <xacro:macro name="cage_wheel" params="name x y">
     <link name="${name}_link">
+      <inertial>
+        <mass value="$(arg wheel_mass)"/>
+        <origin xyz="0 0 0" rpy="0 0 0"/>
+        <inertia ixx="${wheel_transverse_inertia}" ixy="0" ixz="0" iyy="${wheel_axial_inertia}" iyz="0" izz="${wheel_transverse_inertia}"/>
+      </inertial>
       <visual><origin rpy="1.57079632679 0 0"/><geometry><cylinder radius="${wheel_radius_value}" length="$(arg wheel_width)"/></geometry><material name="cage_wheel_gray"/></visual>
       <collision><origin rpy="1.57079632679 0 0"/><geometry><cylinder radius="${wheel_radius_value}" length="$(arg wheel_width)"/></geometry></collision>
     </link>
-    <joint name="base_link_to_${name}" type="fixed">
+    <joint name="base_link_to_${name}" type="continuous">
       <parent link="base_link"/><child link="${name}_link"/>
       <origin xyz="${x} ${y} ${-body_center_z_value + wheel_radius_value}"/>
+      <axis xyz="0 1 0"/>
+      <dynamics damping="$(arg wheel_joint_damping)" friction="$(arg wheel_joint_friction)"/>
     </joint>
   </xacro:macro>
@@ -56,3 +74,31 @@
   <link name="downward_camera_link"/>
   <joint name="base_link_to_downward_camera_link" type="fixed"><parent link="base_link"/><child link="downward_camera_link"/><origin xyz="0.30 0 ${-0.5 * float(xacro.arg('body_height'))}" rpy="0 1.20 0"/></joint>
+  <gazebo>
+    <plugin filename="libignition-gazebo-joint-state-publisher-system.so"
+            name="ignition::gazebo::systems::JointStatePublisher">
+      <topic>/rice_weeding/simulation/wheel_joint_states</topic>
+      <joint_name>base_link_to_front_left_wheel</joint_name>
+      <joint_name>base_link_to_rear_left_wheel</joint_name>
+      <joint_name>base_link_to_front_right_wheel</joint_name>
+      <joint_name>base_link_to_rear_right_wheel</joint_name>
+    </plugin>
+    <plugin filename="libignition-gazebo-diff-drive-system.so"
+            name="ignition::gazebo::systems::DiffDrive">
+      <left_joint>base_link_to_front_left_wheel</left_joint>
+      <left_joint>base_link_to_rear_left_wheel</left_joint>
+      <right_joint>base_link_to_front_right_wheel</right_joint>
+      <right_joint>base_link_to_rear_right_wheel</right_joint>
+      <wheel_separation>$(arg track_width)</wheel_separation>
+      <wheel_radius>${wheel_radius_value}</wheel_radius>
+      <topic>/rice_weeding/simulation/internal/locked_cmd_vel</topic>
+      <odom_topic>/rice_weeding/simulation/internal/diff_drive_odometry</odom_topic>
+      <tf_topic>/rice_weeding/simulation/internal/diff_drive_tf</tf_topic>
+      <max_linear_velocity>$(arg max_forward_velocity)</max_linear_velocity>
+      <min_linear_velocity>-${float(xacro.arg('max_reverse_velocity'))}</min_linear_velocity>
+      <max_angular_velocity>$(arg max_angular_velocity)</max_angular_velocity>
+      <min_angular_velocity>-${float(xacro.arg('max_angular_velocity'))}</min_angular_velocity>
+      <max_linear_acceleration>$(arg max_linear_acceleration)</max_linear_acceleration>
+      <min_linear_acceleration>-${float(xacro.arg('max_linear_deceleration'))}</min_linear_acceleration>
+    </plugin>
+  </gazebo>
 </robot>
